Commit message: fixed simulation issues

File: cbf/franka_description/end_effectors/common/franka_hand.xacro (robot description, xacro)
@@ -126,5 +126,5 @@
       <axis xyz="0 1 0" />
       <limit effort="100" lower="0.0" upper="0.04" velocity="0.2" />
-      <mimic joint="${ee_prefix}finger_joint1" />
+      <!-- no <mimic>: crashes robot_state_publisher 3.4.3 / kdl_parser 2.12.1 on ROS 2 Kilted -->
       <dynamics damping="0.3" />
     </joint>

File: cbf/franka_description/robots/fer/fer.urdf (robot description, URDF)
Before this commit: robot fer, 14 links, 13 joints
Joints:
- joint fer_finger_joint2: mimic joint=fer_finger_joint1 -> (none)
